File: Controlador Cubetto/cubetto_1.brd (EAGLE design)
At the start: 210 x 300 mm, 128 parts

Commit message: update placa
Routing:
- net VCC: track 1241.4 -> 1288.6 mm
- net GND: track 1127.0 -> 1137.8 mm
- net N$114: track 19.8 -> 18.2 mm
- net N$90: track 169.9 -> 168.7 mm
- net N$95: track 51.8 -> 53.1 mm
- net N$93: track 158.5 -> 159.8 mm
- net N$92: track 197.7 -> 196.4 mm
- net N$88: track 129.1 -> 127.9 mm
- net N$86: track 87.2 -> 85.9 mm
- net N$84: track 60.9 -> 59.6 mm
- net N$82: track 21.2 -> 20.0 mm
- net N$30: track 105.4 -> 104.2 mm
- net N$126: track 106.5 -> 105.3 mm
- net N$124: track 196.3 -> 195.0 mm
- net N$122: track 168.5 -> 167.2 mm
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